Commit message: irobot_new添加完成

File: src/irobot_mujoco/asset/urdf/irobot.urdf (robot description, URDF)
Before this commit: robot irobot, 21 links, 20 joints
Links:
- removed link link1_L
- removed link link1_R
- removed link link2_L
- removed link link2_R
- removed link link3_L
- removed link link3_R
- removed link link4_L
- removed link link4_R
- removed link link5_L
- removed link link5_R
- removed link link6_L
- removed link link6_R
- removed link link7_L
- removed link link7_R
- removed link link_clip1_L
- removed link link_clip1_R
- removed link link_clip2_L
- removed link link_clip2_R
- removed link link_neck1
- removed link link_neck2
- added link head_link1, mass 0.0519399235563418; collision mesh filename=package://irobot_description/meshes/head_link1.STL; visual mesh filename=package://irobot_description/meshes/head_link1.STL
- added link head_link2, mass 0.208098890341154; collision mesh filename=package://irobot_description/meshes/head_link2.STL; visual mesh filename=package://irobot_description/meshes/head_link2.STL
- added link head_link3, mass 30.6136843115723
- added link left_arm_link1, mass 0.111538042947354; collision mesh filename=package://irobot_description/meshes/left_arm_link1.STL; visual mesh filename=package://irobot_description/meshes/left_arm_link1.STL
- added link left_arm_link2, mass 0.165341819684868; collision mesh filename=package://irobot_description/meshes/left_arm_link2.STL; visual mesh filename=package://irobot_description/meshes/left_arm_link2.STL
- added link left_arm_link3, mass 0.320011699745351; collision mesh filename=package://irobot_description/meshes/left_arm_link3.STL; visual mesh filename=package://irobot_description/meshes/left_arm_link3.STL
- added link left_arm_link4, mass 0.117835638004833; collision mesh filename=package://irobot_description/meshes/left_arm_link4.STL; visual mesh filename=package://irobot_description/meshes/left_arm_link4.STL
- added link left_arm_link5, mass 0.174906129247525; collision mesh filename=package://irobot_description/meshes/left_arm_link5.STL; visual mesh filename=package://irobot_description/meshes/left_arm_link5.STL
- added link left_arm_link6, mass 0.0486001428262173; collision mesh filename=package://irobot_description/meshes/left_arm_link6.STL; visual mesh filename=package://irobot_description/meshes/left_arm_link6.STL
- added link left_arm_link7, mass 0.0870256121526239; collision mesh filename=package://irobot_description/meshes/left_arm_link7.STL; visual mesh filename=package://irobot_description/meshes/left_arm_link7.STL
- added link left_arm_link8, mass 0.0001
- added link left_hand_link1, mass 0.0470486318704618; collision mesh filename=package://irobot_description/meshes/left_hand_link1.STL; visual mesh filename=package://irobot_description/meshes/left_hand_link1.STL
- added link left_hand_link2, mass 0.0442819627175458; collision mesh filename=package://irobot_description/meshes/left_hand_link2.STL; visual mesh filename=package://irobot_description/meshes/left_hand_link2.STL
- added link right_arm_link1, mass 0.111538042947357; collision mesh filename=package://irobot_description/meshes/right_arm_link1.STL; visual mesh filename=package://irobot_description/meshes/right_arm_link1.STL
- added link right_arm_link2, mass 0.165338288271136; collision mesh filename=package://irobot_description/meshes/right_arm_link2.STL; visual mesh filename=package://irobot_description/meshes/right_arm_link2.STL
- added link right_arm_link3, mass 0.320011699259806; collision mesh filename=package://irobot_description/meshes/right_arm_link3.STL; visual mesh filename=package://irobot_description/meshes/right_arm_link3.STL
- added link right_arm_link4, mass 0.117835638004831; collision mesh filename=package://irobot_description/meshes/right_arm_link4.STL; visual mesh filename=package://irobot_description/meshes/right_arm_link4.STL
- added link right_arm_link5, mass 0.174905784633858; collision mesh filename=package://irobot_description/meshes/right_arm_link5.STL; visual mesh filename=package://irobot_description/meshes/right_arm_link5.STL
- added link right_arm_link6, mass 0.0486001428262178; collision mesh filename=package://irobot_description/meshes/right_arm_link6.STL; visual mesh filename=package://irobot_description/meshes/right_arm_link6.STL
- added link right_arm_link7, mass 0.0870256108294335; collision mesh filename=package://irobot_description/meshes/right_arm_link7.STL; visual mesh filename=package://irobot_description/meshes/right_arm_link7.STL
- added link right_arm_link8, mass 0.0001
- added link right_hand_link1, mass 0.047048635404105; collision mesh filename=package://irobot_description/meshes/right_hand_link1.STL; visual mesh filename=package://irobot_description/meshes/right_hand_link1.STL
- added link right_hand_link2, mass 0.0442819350381612; collision mesh filename=package://irobot_description/meshes/right_hand_link2.STL; visual mesh filename=package://irobot_description/meshes/right_hand_link2.STL
- link base_link: mass 8.9781 -> 27.3425503962047
Joints:
- removed joint joint1_L
- removed joint joint1_R
- removed joint joint2_L
- removed joint joint2_R
- removed joint joint3_L
- removed joint joint3_R
- removed joint joint4_L
- removed joint joint4_R
- removed joint joint5_L
- removed joint joint5_R
- removed joint joint6_L
- removed joint joint6_R
- removed joint joint7_L
- removed joint joint7_R
- removed joint joint_clip1_L
- removed joint joint_clip1_R
- removed joint joint_clip2_L
- removed joint joint_clip2_R
- removed joint joint_neck1
- removed joint joint_neck2
- added joint head_joint1: type revolute, parent base_link, child head_link1, origin xyz=0 0 1.5945 rpy=0 0 0, axis 0 0 1, limit lower=-3.14 upper=3.14 effort=0 velocity=0
- added joint head_joint2: type revolute, parent head_link1, child head_link2, origin xyz=0 0 0 rpy=0 0 0, axis 0 1 0, limit lower=-3.14 upper=3.14 effort=0 velocity=0
- added joint head_joint3: type fixed, parent head_link2, child head_link3, origin xyz=0.079721 0 0.029759 rpy=0 0 0, axis 0 0 0
- added joint left_arm_joint1: type revolute, parent base_link, child left_arm_link1, origin xyz=0 0.159 1.45 rpy=0 0 0, axis 0 1 0, limit lower=-3.14 upper=3.14 effort=0 velocity=0
- added joint left_arm_joint2: type revolute, parent left_arm_link1, child left_arm_link2, origin xyz=0 0 0 rpy=0 0 0, axis -1 0 0, limit lower=-3.14 upper=3.14 effort=0 velocity=0
- added joint left_arm_joint3: type revolute, parent left_arm_link2, child left_arm_link3, origin xyz=0 0 -0.27 rpy=0 0 0, axis 0 0 -1, limit lower=-3.14 upper=3.14 effort=0 velocity=0
- added joint left_arm_joint4: type revolute, parent left_arm_link3, child left_arm_link4, origin xyz=0 0 0 rpy=0 0 0, axis 0 -1 0, limit lower=-3.14 upper=3.14 effort=0 velocity=0
- added joint left_arm_joint5: type revolute, parent left_arm_link4, child left_arm_link5, origin xyz=0 0 -0.24 rpy=0 0 0, axis 0 0 -1, limit lower=-3.14 upper=3.14 effort=0 velocity=0
- added joint left_arm_joint6: type revolute, parent left_arm_link5, child left_arm_link6, origin xyz=0 0 0 rpy=0 0 0, axis 0 -1 0, limit lower=-3.14 upper=3.14 effort=0 velocity=0
- added joint left_arm_joint7: type revolute, parent left_arm_link6, child left_arm_link7, origin xyz=0 0 -0.042 rpy=0 0 0, axis 0 0 1, limit lower=-3.14 upper=3.14 effort=0 velocity=0
- added joint left_arm_joint8: type fixed, parent left_arm_link7, child left_arm_link8, origin xyz=0 0 -0.1 rpy=0 1.5708 0, axis 0 0 1, limit lower=-3.14 upper=3.14 effort=0 velocity=0
- added joint left_hand_joint1: type revolute, parent left_arm_link7, child left_hand_link1, origin xyz=0 -0.018 -0.037 rpy=0 0 0, axis 1 0 0, limit lower=-3.14 upper=3.14 effort=0 velocity=0
- added joint left_hand_joint2: type revolute, parent left_arm_link7, child left_hand_link2, origin xyz=0 0.018 -0.037 rpy=0 0 0, axis 1 0 0, limit lower=-3.14 upper=3.14 effort=0 velocity=0
- added joint right_arm_joint1: type revolute, parent base_link, child right_arm_link1, origin xyz=0 -0.16 1.45 rpy=0 0 0, axis 0 -1 0, limit lower=-3.14 upper=3.14 effort=0 velocity=0
- added joint right_arm_joint2: type revolute, parent right_arm_link1, child right_arm_link2, origin xyz=0 0 0 rpy=0 0 0, axis -1 0 0, limit lower=-3.14 upper=3.14 effort=0 velocity=0
- added joint right_arm_joint3: type revolute, parent right_arm_link2, child right_arm_link3, origin xyz=0 0 -0.27 rpy=0 0 0, axis 0 0 -1, limit lower=-3.14 upper=3.14 effort=0 velocity=0
- added joint right_arm_joint4: type revolute, parent right_arm_link3, child right_arm_link4, origin xyz=0 0 0 rpy=0 0 0, axis 0 -1 0, limit lower=-3.14 upper=3.14 effort=0 velocity=0
- added joint right_arm_joint5: type revolute, parent right_arm_link4, child right_arm_link5, origin xyz=0 0 -0.24 rpy=0 0 0, axis 0 0 -1, limit lower=-3.14 upper=3.14 effort=0 velocity=0
- added joint right_arm_joint6: type revolute, parent right_arm_link5, child right_arm_link6, origin xyz=0 0 0 rpy=0 0 0, axis 0 1 0, limit lower=-3.14 upper=3.14 effort=0 velocity=0
- added joint right_arm_joint7: type revolute, parent right_arm_link6, child right_arm_link7, origin xyz=0 0 -0.042 rpy=0 0 0, axis 0 0 1, limit lower=-3.14 upper=3.14 effort=0 velocity=0
- added joint right_arm_joint8: type fixed, parent right_arm_link7, child right_arm_link8, origin xyz=0 0 -0.1 rpy=0 1.5708 0, axis 0 0 1, limit lower=-3.14 upper=3.14 effort=0 velocity=0
- added joint right_hand_joint1: type revolute, parent right_arm_link7, child right_hand_link1, origin xyz=0 0.018 -0.037 rpy=0 0 0, axis 1 0 0, limit lower=-3.14 upper=3.14 effort=0 velocity=0
- added joint right_hand_joint2: type revolute, parent right_arm_link7, child right_hand_link2, origin xyz=0 -0.018 -0.037 rpy=0 0 0, axis 1 0 0, limit lower=-3.14 upper=3.14 effort=0 velocity=0
