Commit message: 添加方块搭建轨迹

File: src/irobot_description/urdf/irobot_visual.urdf (robot description, URDF)
Before this commit: robot irobot, 24 links, 23 joints
Links:
- removed link right_arm_link7
- removed link right_arm_link8
- removed link right_hand_link1
- removed link right_hand_link2
- added link clipbase_link, mass 0.0676692041651645; collision mesh filename=../meshes/clipbase_link.STL; visual mesh filename=../meshes/clipbase_link.STL
- added link joint_Link1_1, mass 0.0244077119794162; collision mesh filename=../meshes/joint_Link1_1.STL; visual mesh filename=../meshes/joint_Link1_1.STL
- added link joint_link1_2, mass 0.0825284444858284; collision mesh filename=../meshes/joint_link1_2.STL; visual mesh filename=../meshes/joint_link1_2.STL
- added link joint_link2_1, mass 0.0249594770057966; collision mesh filename=../meshes/joint_link2_1.STL; visual mesh filename=../meshes/joint_link2_1.STL
- added link joint_link2_2, mass 0.0825284444858284; collision mesh filename=../meshes/joint_link2_2.STL; visual mesh filename=../meshes/joint_link2_2.STL
Joints:
- removed joint right_arm_joint8
- removed joint right_hand_joint1
- removed joint right_hand_joint2
- added joint joint1_1: type continuous, parent clipbase_link, child joint_Link1_1, origin xyz=0.0470000000004201 -0.0179999999999996 -0.0430000000000004 rpy=0 0 0, axis 1 0 0
- added joint joint1_2: type continuous, parent joint_Link1_1, child joint_link1_2, origin xyz=-0.00700000000000021 -0.00699839115061319 -0.0464760424445006 rpy=0 0 0, axis 1 0 0
- added joint joint2_1: type continuous, parent clipbase_link, child joint_link2_1, origin xyz=0.0470000000004201 0.0179999999999995 -0.0430000000000001 rpy=0 0 0, axis 1 0 0
- added joint joint2_2: type continuous, parent joint_link2_1, child joint_link2_2, origin xyz=-0.00700000000000003 0.00704396779938812 -0.0464691566271775 rpy=0 0 0, axis 1 0 0
- joint right_arm_joint7: axis 0 0 1 -> 0 1 0; child right_arm_link7 -> clipbase_link; origin xyz=0 0 -0.042 rpy=0 0 0 -> xyz=0 0 -0.036 rpy=0 0 0
